Commit message: control pitch angle

File: lidar_with_mirror_description/urdf/orne_box_lidar_with_mirror.gazebo.xacro (robot description, xacro)
@@ -93,5 +93,5 @@
         <scan>
           <horizontal>
-            <samples>682</samples>
+            <samples>341</samples>
             <resolution>1</resolution>
             <min_angle>${-PI/180*60}</min_angle>
@@ -100,7 +100,7 @@
         </scan>
         <range>
-          <min>0.10</min>
+          <min>0.06</min>
           <max>5.60</max>
-          <resolution>0.01</resolution>
+          <resolution>0.001</resolution>
         </range>
         <noise>
@@ -128,5 +128,5 @@
         <scan>
           <horizontal>
-            <samples>341</samples>
+            <samples>170</samples>
             <resolution>1</resolution>
             <min_angle>${PI/180*60}</min_angle>
@@ -135,7 +135,7 @@
         </scan>
         <range>
-          <min>0.10</min>
+          <min>0.06</min>
           <max>5.60</max>
-          <resolution>0.01</resolution>
+          <resolution>0.001</resolution>
         </range>
         <noise>
@@ -163,5 +163,5 @@
         <scan>
           <horizontal>
-            <samples>341</samples>
+            <samples>170</samples>
             <resolution>1</resolution>
             <min_angle>${-PI/180*120}</min_angle>
@@ -170,7 +170,7 @@
         </scan>
         <range>
-          <min>0.10</min>
+          <min>0.06</min>
           <max>5.60</max>
-          <resolution>0.01</resolution>
+          <resolution>0.001</resolution>
         </range>
         <noise>

File: lidar_with_mirror_description/urdf/orne_box_lidar_with_mirror.urdf.xacro (robot description, xacro)
@@ -138,8 +138,10 @@
     </inertial>
   </link>
-  <joint name="caster_front_joint" type="fixed">
+  <joint name="caster_front_joint" type="prismatic">
     <parent link="base_link"/>
     <child link="caster_front_link"/>
     <origin xyz="0.362 0 0.050" rpy="0 0 0"/>
+    <axis xyz="0 0 1"/>
+    <limit effort="100" velocity="100.0" lower="-1" upper="1" />
   </joint>
   <link name="caster_front_link">
@@ -335,5 +337,15 @@
       <hardwareInterface>hardware_interface/PositionJointInterface</hardwareInterface>
     </joint>
-  <actuator name="lidar_with_mirror_prismatic_joint">
+  <actuator name="lidar_with_mirror_prismatic_motor">
+      <hardwareInterface>hardware_interface/PositionJointInterface</hardwareInterface>
+      <mechanicalReduction>1</mechanicalReduction>
+    </actuator>
+  </transmission>
+  <transmission name="tran8">
+    <type>transmission_interface/SimpleTransmission</type>
+    <joint name="caster_front_joint">
+      <hardwareInterface>hardware_interface/PositionJointInterface</hardwareInterface>
+    </joint>
+  <actuator name="caster_front_motor">
       <hardwareInterface>hardware_interface/PositionJointInterface</hardwareInterface>
       <mechanicalReduction>1</mechanicalReduction>

Commit message: check correction

File: lidar_with_mirror_description/urdf/orne_box_lidar_with_mirror.gazebo.xacro (robot description, xacro)
@@ -100,5 +100,5 @@
         </scan>
         <range>
-          <min>0.06</min>
+          <min>0.10</min>
           <max>5.60</max>
           <resolution>0.001</resolution>
@@ -135,5 +135,5 @@
         </scan>
         <range>
-          <min>0.06</min>
+          <min>0.10</min>
           <max>5.60</max>
           <resolution>0.001</resolution>
@@ -170,5 +170,5 @@
         </scan>
         <range>
-          <min>0.06</min>
+          <min>0.10</min>
           <max>5.60</max>
           <resolution>0.001</resolution>

File: lidar_with_mirror_description/urdf/orne_box_lidar_with_mirror.urdf.xacro (robot description, xacro)
@@ -42,4 +42,5 @@
       <material name="orange"/>
     </visual>
+<!--
     <collision>
       <origin xyz="0.090 0 0.1715" rpy="0 0 0"/>
@@ -66,4 +67,5 @@
       </geometry>
     </collision>
+-->
     <inertial>
       <origin xyz="0.090 0 0.1715" rpy="0 0 0"/>
@@ -72,8 +74,22 @@
     </inertial>
   </link>
+  <joint name="wheel_hinge" type="revolute">
+    <parent link="base_link"/>
+    <child link="wheel_link"/>
+    <origin xyz="0.0 0.0 0.152" rpy="0 0 0"/>
+    <axis xyz="1 0 0"/>
+    <limit effort="100" velocity="100.0"  lower="-5000" upper="5000" />
+  </joint>
+  <link name="wheel_link">
+    <inertial>
+      <origin xyz="0 0 0" />
+      <mass value="0.2" />
+      <inertia ixx="0.1" ixy="0.0" ixz="0.0" iyy="0.1" iyz="0.0" izz="0.1" />
+    </inertial>
+  </link>
   <joint name="left_wheel_hinge" type="revolute">
-    <parent link="base_link"/>
+    <parent link="wheel_link"/>
     <child link="wheel_left_link"/>
-    <origin xyz="0.0 0.23075 0.152" rpy="${-PI/2} 0 0"/>
+    <origin xyz="0.0 0.23075 0.0" rpy="${-PI/2} 0 0"/>
     <axis xyz="0 0 1"/>
     <limit effort="100" velocity="100.0"  lower="-5000" upper="5000" />
@@ -106,7 +122,7 @@
   </link>
   <joint name="right_wheel_hinge" type="revolute">
-    <parent link="base_link"/>
+    <parent link="wheel_link"/>
     <child link="wheel_right_link"/>
-    <origin xyz="0.0 -0.23075 0.152" rpy="${-PI/2} 0 0"/>
+    <origin xyz="0.0 -0.23075 0.0" rpy="${-PI/2} 0 0"/>
     <axis xyz="0 0 1"/>
     <limit effort="100" velocity="100.0"  lower="-5000" upper="5000" />
@@ -239,5 +255,5 @@
     <parent link="lidar_with_mirror_center_link"/>
     <child link="lidar_with_mirror_mirror1_roll_link"/>
-    <origin xyz="0 ${len} 0" rpy="${-PI/2} 0 0"/>
+    <origin xyz="0 ${len} 0" rpy="${-PI/4} 0 0"/>
     <axis xyz="-1 0 0"/>
     <limit effort="100" velocity="100.0" lower="${-PI}" upper="${PI}" />
@@ -257,5 +273,5 @@
     <parent link="lidar_with_mirror_center_link"/>
     <child link="lidar_with_mirror_mirror2_roll_link"/>
-    <origin xyz="0 ${-len} 0" rpy="${PI/2} 0 0"/>
+    <origin xyz="0 ${-len} 0" rpy="${PI/4} 0 0"/>
     <axis xyz="1 0 0"/>
     <limit effort="100" velocity="100.0" lower="${-PI}" upper="${PI}" />
@@ -352,3 +368,13 @@
     </actuator>
   </transmission>
+  <transmission name="tran9">
+    <type>transmission_interface/SimpleTransmission</type>
+    <joint name="wheel_hinge">
+      <hardwareInterface>hardware_interface/PositionJointInterface</hardwareInterface>
+    </joint>
+  <actuator name="wheel_hinge_motor">
+      <hardwareInterface>hardware_interface/PositionJointInterface</hardwareInterface>
+      <mechanicalReduction>1</mechanicalReduction>
+    </actuator>
+  </transmission>
 </robot>

Commit message: upside down

File: lidar_with_mirror_description/urdf/orne_box_lidar_with_mirror.gazebo.xacro (robot description, xacro)
@@ -130,6 +130,6 @@
             <samples>170</samples>
             <resolution>1</resolution>
-            <min_angle>${PI/180*60}</min_angle>
-            <max_angle>${PI/180*120}</max_angle>
+            <min_angle>${-PI/180*120}</min_angle>
+            <max_angle>${-PI/180*60}</max_angle>
           </horizontal>
         </scan>
@@ -165,6 +165,6 @@
             <samples>170</samples>
             <resolution>1</resolution>
-            <min_angle>${-PI/180*120}</min_angle>
-            <max_angle>${-PI/180*60}</max_angle>
+            <min_angle>${PI/180*60}</min_angle>
+            <max_angle>${PI/180*120}</max_angle>
           </horizontal>
         </scan>

File: lidar_with_mirror_description/urdf/orne_box_lidar_with_mirror.urdf.xacro (robot description, xacro)
@@ -234,5 +234,5 @@
     <parent link="lidar_with_mirror_pitch_link"/>
     <child link="lidar_with_mirror_roll_link"/>
-    <origin xyz="0 0 0" rpy="0 0 0"/>
+    <origin xyz="0 0 0" rpy="${PI} 0 0"/>
     <axis xyz="1 0 0"/>
     <limit effort="100" velocity="100.0" lower="${-PI}" upper="${PI}" />
@@ -283,6 +283,6 @@
     <parent link="lidar_with_mirror_mirror1_yaw_link"/>
     <child link="lidar_with_mirror_mirror1_roll_link"/>
-    <origin xyz="0 0 0" rpy="${-PI/4} 0 0"/>
-    <axis xyz="-1 0 0"/>
+    <origin xyz="0 0 0" rpy="${PI/4} 0 0"/>
+    <axis xyz="1 0 0"/>
     <limit effort="100" velocity="100.0" lower="${-PI}" upper="${PI}" />
   </joint>
@@ -309,5 +309,5 @@
   </link>
   <xacro:include filename="$(find icart_mini_description)/urdf/sensors/hokuyo.urdf.xacro"/>
-  <xacro:sensor_hokuyo name="lidar_with_mirror_left" parent="lidar_with_mirror_mirror1_prismatic2_link">
+  <xacro:sensor_hokuyo name="lidar_with_mirror_right" parent="lidar_with_mirror_mirror1_prismatic2_link">
     <origin xyz="0 0 0" rpy="0 0 0"/>
   </xacro:sensor_hokuyo>
@@ -343,6 +343,6 @@
     <parent link="lidar_with_mirror_mirror2_yaw_link"/>
     <child link="lidar_with_mirror_mirror2_roll_link"/>
-    <origin xyz="0 0 0" rpy="${PI/4} 0 0"/>
-    <axis xyz="1 0 0"/>
+    <origin xyz="0 0 0" rpy="${-PI/4} 0 0"/>
+    <axis xyz="-1 0 0"/>
     <limit effort="100" velocity="100.0" lower="${-PI}" upper="${PI}" />
   </joint>
@@ -369,5 +369,5 @@
   </link>
   <xacro:include filename="$(find icart_mini_description)/urdf/sensors/hokuyo.urdf.xacro"/>
-  <xacro:sensor_hokuyo name="lidar_with_mirror_right" parent="lidar_with_mirror_mirror2_prismatic2_link">
+  <xacro:sensor_hokuyo name="lidar_with_mirror_left" parent="lidar_with_mirror_mirror2_prismatic2_link">
     <origin xyz="0 0 0" rpy="0 0 0"/>
   </xacro:sensor_hokuyo>
