Commit message: for video

File: lidar_with_mirror_description/urdf/lidar_with_mirror.urdf.xacro (robot description, xacro)
@@ -27,10 +27,23 @@
     </inertial>
   </link>
-  <xacro:property name="len" value="0.1" />
+  <xacro:property name="len" value="0.06" />
   <xacro:property name="front" value="0" />
   <xacro:property name="height" value="0.3" />
+  <joint name="laser_joint" type="fixed">
+    <parent link="lidar_with_mirror_prismatic_link"/>
+    <child link="laser"/>
+    <origin xyz="${front} 0 ${height}" rpy="0 ${PI/9} 0"/>
+    <axis xyz="1 0 0"/>
+  </joint>
+  <link name="laser">
+    <inertial>
+      <origin xyz="0 0 0" />
+      <mass value="0.2" />
+      <inertia ixx="0.1" ixy="0.0" ixz="0.0" iyy="0.1" iyz="0.0" izz="0.1" />
+    </inertial>
+  </link>
   <xacro:include filename="$(find icart_mini_description)/urdf/sensors/hokuyo.urdf.xacro"/>
   <xacro:sensor_hokuyo name="lidar_with_mirror_center" parent="lidar_with_mirror_prismatic_link">
-    <origin xyz="${front} 0 ${height}" rpy="0 ${PI/9} 0"/>
+    <origin xyz="${front} 0 ${height}" rpy="0 0 0"/>
   </xacro:sensor_hokuyo>
   <joint name="lidar_with_mirror_mirror1_roll_joint" type="fixed">
@@ -48,6 +61,19 @@
     </inertial>
   </link>
+  <joint name="lidar_with_mirror_mirror1_pitch_joint" type="fixed">
+    <parent link="lidar_with_mirror_mirror1_roll_link"/>
+    <child link="lidar_with_mirror_mirror1_pitch_link"/>
+    <origin xyz="0 0 0" rpy="0 0 0"/>
+    <axis xyz="0 0 -1"/>
+  </joint>
+  <link name="lidar_with_mirror_mirror1_pitch_link">
+    <inertial>
+      <origin xyz="0 0 0" />
+      <mass value="0.2" />
+      <inertia ixx="0.1" ixy="0.0" ixz="0.0" iyy="0.1" iyz="0.0" izz="0.1" />
+    </inertial>
+  </link>
   <xacro:include filename="$(find icart_mini_description)/urdf/sensors/hokuyo.urdf.xacro"/>
-  <xacro:sensor_hokuyo name="lidar_with_mirror_left" parent="lidar_with_mirror_mirror1_roll_link">
+  <xacro:sensor_hokuyo name="lidar_with_mirror_left" parent="lidar_with_mirror_mirror1_pitch_link">
     <origin xyz="0 ${-len} 0" rpy="0 0 0"/>
   </xacro:sensor_hokuyo>

Commit message: simulation

File: lidar_with_mirror_description/urdf/lidar_with_mirror.urdf.xacro (robot description, xacro)
@@ -114,5 +114,5 @@
     <limit effort="100" velocity="100.0" lower="${-PI}" upper="${PI}" />
   </joint>
-  <link name="lidar_with_mirror_mirror2_roll_link">
+  <link name="${name}_mirror2_roll_link">
     <inertial>
       <origin xyz="0 0 0" />
@@ -139,40 +139,20 @@
     <origin xyz="0 0 0" rpy="0 0 0"/>
   </xacro:sensor_hokuyo>
+  <transmission name="tran5">
+    <type>transmission_interface/SimpleTransmission</type>
+    <joint name="${name}_mirror1_roll_joint">
+      <hardwareInterface>hardware_interface/PositionJointInterface</hardwareInterface>
+    </joint>
+  <actuator name="${name}_mirror1_roll_motor">
+      <hardwareInterface>hardware_interface/PositionJointInterface</hardwareInterface>
+      <mechanicalReduction>1</mechanicalReduction>
+    </actuator>
+  </transmission>
   <transmission name="tran6">
     <type>transmission_interface/SimpleTransmission</type>
-    <joint name="lidar_with_mirror_mirror2_roll_joint">
-      <hardwareInterface>hardware_interface/PositionJointInterface</hardwareInterface>
-    </joint>
-  <actuator name="lidar_with_mirror_mirror2_roll_motor">
-      <hardwareInterface>hardware_interface/PositionJointInterface</hardwareInterface>
-      <mechanicalReduction>1</mechanicalReduction>
-    </actuator>
-  </transmission>
-  <transmission name="tran7">
-    <type>transmission_interface/SimpleTransmission</type>
-    <joint name="lidar_with_mirror_prismatic_joint">
-      <hardwareInterface>hardware_interface/PositionJointInterface</hardwareInterface>
-    </joint>
-  <actuator name="lidar_with_mirror_prismatic_motor">
-      <hardwareInterface>hardware_interface/PositionJointInterface</hardwareInterface>
-      <mechanicalReduction>1</mechanicalReduction>
-    </actuator>
-  </transmission>
-  <transmission name="tran8">
-    <type>transmission_interface/SimpleTransmission</type>
-    <joint name="caster_front_joint">
-      <hardwareInterface>hardware_interface/PositionJointInterface</hardwareInterface>
-    </joint>
-  <actuator name="caster_front_motor">
-      <hardwareInterface>hardware_interface/PositionJointInterface</hardwareInterface>
-      <mechanicalReduction>1</mechanicalReduction>
-    </actuator>
-  </transmission>
-  <transmission name="tran9">
-    <type>transmission_interface/SimpleTransmission</type>
-    <joint name="wheel_hinge">
-      <hardwareInterface>hardware_interface/PositionJointInterface</hardwareInterface>
-    </joint>
-  <actuator name="wheel_hinge_motor">
+    <joint name="${name}_mirror2_roll_joint">
+      <hardwareInterface>hardware_interface/PositionJointInterface</hardwareInterface>
+    </joint>
+  <actuator name="${name}_mirror2_roll_motor">
       <hardwareInterface>hardware_interface/PositionJointInterface</hardwareInterface>
       <mechanicalReduction>1</mechanicalReduction>
@@ -181,8 +161,8 @@
   <transmission name="tran10">
     <type>transmission_interface/SimpleTransmission</type>
-    <joint name="lidar_with_mirror_mirror1_prismatic_joint">
-      <hardwareInterface>hardware_interface/PositionJointInterface</hardwareInterface>
-    </joint>
-    <actuator name="lidar_with_mirror_mirror1_prismatic_motor">
+    <joint name="${name}_mirror1_prismatic_joint">
+      <hardwareInterface>hardware_interface/PositionJointInterface</hardwareInterface>
+    </joint>
+    <actuator name="${name}_mirror1_prismatic_motor">
       <hardwareInterface>hardware_interface/PositionJointInterface</hardwareInterface>
       <mechanicalReduction>1</mechanicalReduction>
@@ -191,8 +171,8 @@
   <transmission name="tran11">
     <type>transmission_interface/SimpleTransmission</type>
-    <joint name="lidar_with_mirror_mirror2_prismatic_joint">
-      <hardwareInterface>hardware_interface/PositionJointInterface</hardwareInterface>
-    </joint>
-    <actuator name="lidar_with_mirror_mirror2_prismatic_motor">
+    <joint name="${name}_mirror2_prismatic_joint">
+      <hardwareInterface>hardware_interface/PositionJointInterface</hardwareInterface>
+    </joint>
+    <actuator name="${name}_mirror2_prismatic_motor">
       <hardwareInterface>hardware_interface/PositionJointInterface</hardwareInterface>
       <mechanicalReduction>1</mechanicalReduction>
@@ -201,8 +181,8 @@
   <transmission name="tran12">
     <type>transmission_interface/SimpleTransmission</type>
-    <joint name="lidar_with_mirror_mirror1_prismatic2_joint">
-      <hardwareInterface>hardware_interface/PositionJointInterface</hardwareInterface>
-    </joint>
-    <actuator name="lidar_with_mirror_mirror1_prismatic2_motor">
+    <joint name="${name}_mirror1_prismatic2_joint">
+      <hardwareInterface>hardware_interface/PositionJointInterface</hardwareInterface>
+    </joint>
+    <actuator name="${name}_mirror1_prismatic2_motor">
       <hardwareInterface>hardware_interface/PositionJointInterface</hardwareInterface>
       <mechanicalReduction>1</mechanicalReduction>
@@ -211,8 +191,8 @@
   <transmission name="tran13">
     <type>transmission_interface/SimpleTransmission</type>
-    <joint name="lidar_with_mirror_mirror2_prismatic2_joint">
-      <hardwareInterface>hardware_interface/PositionJointInterface</hardwareInterface>
-    </joint>
-    <actuator name="lidar_with_mirror_mirror2_prismatic2_motor">
+    <joint name="${name}_mirror2_prismatic2_joint">
+      <hardwareInterface>hardware_interface/PositionJointInterface</hardwareInterface>
+    </joint>
+    <actuator name="${name}_mirror2_prismatic2_motor">
       <hardwareInterface>hardware_interface/PositionJointInterface</hardwareInterface>
       <mechanicalReduction>1</mechanicalReduction>
@@ -221,8 +201,8 @@
   <transmission name="tran14">
     <type>transmission_interface/SimpleTransmission</type>
-    <joint name="lidar_with_mirror_mirror1_pitch_joint">
-      <hardwareInterface>hardware_interface/PositionJointInterface</hardwareInterface>
-    </joint>
-  <actuator name="lidar_with_mirror_mirror1_pitch_motor">
+    <joint name="${name}_mirror1_pitch_joint">
+      <hardwareInterface>hardware_interface/PositionJointInterface</hardwareInterface>
+    </joint>
+  <actuator name="${name}_mirror1_pitch_motor">
       <hardwareInterface>hardware_interface/PositionJointInterface</hardwareInterface>
       <mechanicalReduction>1</mechanicalReduction>
@@ -231,8 +211,8 @@
   <transmission name="tran15">
     <type>transmission_interface/SimpleTransmission</type>
-    <joint name="lidar_with_mirror_mirror2_pitch_joint">
-      <hardwareInterface>hardware_interface/PositionJointInterface</hardwareInterface>
-    </joint>
-  <actuator name="lidar_with_mirror_mirror2_pitch_motor">
+    <joint name="${name}_mirror2_pitch_joint">
+      <hardwareInterface>hardware_interface/PositionJointInterface</hardwareInterface>
+    </joint>
+  <actuator name="${name}_mirror2_pitch_motor">
       <hardwareInterface>hardware_interface/PositionJointInterface</hardwareInterface>
       <mechanicalReduction>1</mechanicalReduction>

File: lidar_with_mirror_description/urdf/orne_box_lidar_with_mirror.urdf.xacro (robot description, xacro)
@@ -206,5 +206,5 @@
     <parent link="base_link"/>
     <child link="lidar_with_mirror_prismatic_link"/>
-    <origin xyz="1.0 0 0.3" rpy="0 0 0"/>
+    <origin xyz="-0.15 0 0.56" rpy="0 0 0"/>
     <axis xyz="0 0 1"/>
     <limit effort="100" velocity="100.0" lower="-0.3" upper="1" />
@@ -234,5 +234,5 @@
     <parent link="lidar_with_mirror_pitch_link"/>
     <child link="lidar_with_mirror_roll_link"/>
-    <origin xyz="0 0 0" rpy="${PI} 0 0"/>
+    <origin xyz="0 0 0" rpy="0 0 0"/>
     <axis xyz="1 0 0"/>
     <limit effort="100" velocity="100.0" lower="${-PI}" upper="${PI}" />
@@ -245,131 +245,8 @@
     </inertial>
   </link>
-  <xacro:property name="len" value="0.1" />
-  <xacro:property name="front" value="0" />
-  <xacro:property name="height" value="0" />
-  <xacro:include filename="$(find icart_mini_description)/urdf/sensors/hokuyo.urdf.xacro"/>
-  <xacro:sensor_hokuyo name="lidar_with_mirror_center" parent="lidar_with_mirror_roll_link">
-    <origin xyz="${front} 0 ${height}" rpy="0 0 0"/>
-  </xacro:sensor_hokuyo>
-  <joint name="lidar_with_mirror_mirror1_prismatic_joint" type="prismatic">
-    <parent link="lidar_with_mirror_center_link"/>
-    <child link="lidar_with_mirror_mirror1_prismatic_link"/>
-    <origin xyz="0 ${len} 0" rpy="0 0 0"/>
-    <axis xyz="0 1 0"/>
-    <limit effort="100" velocity="100.0" lower="-1" upper="1" />
-  </joint>
-  <link name="lidar_with_mirror_mirror1_prismatic_link">
-    <inertial>
-      <origin xyz="0 0 0" />
-      <mass value="0.01" />
-      <inertia ixx="0.1" ixy="0.0" ixz="0.0" iyy="0.1" iyz="0.0" izz="0.1" />
-    </inertial>
-  </link>
-  <joint name="lidar_with_mirror_mirror1_yaw_joint" type="revolute">
-    <parent link="lidar_with_mirror_mirror1_prismatic_link"/>
-    <child link="lidar_with_mirror_mirror1_yaw_link"/>
+  <xacro:include filename="$(find lidar_with_mirror_description)/urdf/lidar_with_mirror.urdf.xacro" />
+  <xacro:lidar_with_mirror name="lidar_with_mirror" parent="lidar_with_mirror_roll_link" left_roll_rad="0.769999299112962" left_pitch_rad="-0.05" left_distance_m="0.073124500184212" right_roll_rad="0.787426157712581" right_pitch_rad="-0.05" right_distance_m="0.072588298861567">
     <origin xyz="0 0 0" rpy="0 0 0"/>
-    <axis xyz="0 0 1"/>
-    <limit effort="100" velocity="100.0" lower="${-PI}" upper="${PI}" />
-  </joint>
-  <link name="lidar_with_mirror_mirror1_yaw_link">
-    <inertial>
-      <origin xyz="0 0 0" />
-      <mass value="0.01" />
-      <inertia ixx="0.1" ixy="0.0" ixz="0.0" iyy="0.1" iyz="0.0" izz="0.1" />
-    </inertial>
-  </link>
-  <joint name="lidar_with_mirror_mirror1_roll_joint" type="revolute">
-    <parent link="lidar_with_mirror_mirror1_yaw_link"/>
-    <child link="lidar_with_mirror_mirror1_roll_link"/>
-    <origin xyz="0 0 0" rpy="${PI/4} 0 0"/>
-    <axis xyz="1 0 0"/>
-    <limit effort="100" velocity="100.0" lower="${-PI}" upper="${PI}" />
-  </joint>
-  <link name="lidar_with_mirror_mirror1_roll_link">
-    <inertial>
-      <origin xyz="0 0 0" />
-      <mass value="0.01" />
-      <inertia ixx="0.1" ixy="0.0" ixz="0.0" iyy="0.1" iyz="0.0" izz="0.1" />
-    </inertial>
-  </link>
-  <joint name="lidar_with_mirror_mirror1_prismatic2_joint" type="prismatic">
-    <parent link="lidar_with_mirror_mirror1_roll_link"/>
-    <child link="lidar_with_mirror_mirror1_prismatic2_link"/>
-    <origin xyz="0 ${-len} 0" rpy="0 0 0"/>
-    <axis xyz="0 -1 0"/>
-    <limit effort="100" velocity="100.0" lower="-1" upper="1" />
-  </joint>
-  <link name="lidar_with_mirror_mirror1_prismatic2_link">
-    <inertial>
-      <origin xyz="0 0 0" />
-      <mass value="0.01" />
-      <inertia ixx="0.1" ixy="0.0" ixz="0.0" iyy="0.1" iyz="0.0" izz="0.1" />
-    </inertial>
-  </link>
-  <xacro:include filename="$(find icart_mini_description)/urdf/sensors/hokuyo.urdf.xacro"/>
-  <xacro:sensor_hokuyo name="lidar_with_mirror_right" parent="lidar_with_mirror_mirror1_prismatic2_link">
-    <origin xyz="0 0 0" rpy="0 0 0"/>
-  </xacro:sensor_hokuyo>
-  <joint name="lidar_with_mirror_mirror2_prismatic_joint" type="prismatic">
-    <parent link="lidar_with_mirror_center_link"/>
-    <child link="lidar_with_mirror_mirror2_prismatic_link"/>
-    <origin xyz="0 ${-len} 0" rpy="0 0 0"/>
-    <axis xyz="0 -1 0"/>
-    <limit effort="100" velocity="100.0" lower="-1" upper="1" />
-  </joint>
-  <link name="lidar_with_mirror_mirror2_prismatic_link">
-    <inertial>
-      <origin xyz="0 0 0" />
-      <mass value="0.01" />
-      <inertia ixx="0.1" ixy="0.0" ixz="0.0" iyy="0.1" iyz="0.0" izz="0.1" />
-    </inertial>
-  </link>
-  <joint name="lidar_with_mirror_mirror2_yaw_joint" type="revolute">
-    <parent link="lidar_with_mirror_mirror2_prismatic_link"/>
-    <child link="lidar_with_mirror_mirror2_yaw_link"/>
-    <origin xyz="0 0 0" rpy="0 0 0"/>
-    <axis xyz="0 0 1"/>
-    <limit effort="100" velocity="100.0" lower="${-PI}" upper="${PI}" />
-  </joint>
-  <link name="lidar_with_mirror_mirror2_yaw_link">
-    <inertial>
-      <origin xyz="0 0 0" />
-      <mass value="0.01" />
-      <inertia ixx="0.1" ixy="0.0" ixz="0.0" iyy="0.1" iyz="0.0" izz="0.1" />
-    </inertial>
-  </link>
-  <joint name="lidar_with_mirror_mirror2_roll_joint" type="revolute">
-    <parent link="lidar_with_mirror_mirror2_yaw_link"/>
-    <child link="lidar_with_mirror_mirror2_roll_link"/>
-    <origin xyz="0 0 0" rpy="${-PI/4} 0 0"/>
-    <axis xyz="-1 0 0"/>
-    <limit effort="100" velocity="100.0" lower="${-PI}" upper="${PI}" />
-  </joint>
-  <link name="lidar_with_mirror_mirror2_roll_link">
-    <inertial>
-      <origin xyz="0 0 0" />
-      <mass value="0.01" />
-      <inertia ixx="0.1" ixy="0.0" ixz="0.0" iyy="0.1" iyz="0.0" izz="0.1" />
-    </inertial>
-  </link>
-  <joint name="lidar_with_mirror_mirror2_prismatic2_joint" type="prismatic">
-    <parent link="lidar_with_mirror_mirror2_roll_link"/>
-    <child link="lidar_with_mirror_mirror2_prismatic2_link"/>
-    <origin xyz="0 ${len} 0" rpy="0 0 0"/>
-    <axis xyz="0 1 0"/>
-    <limit effort="100" velocity="100.0" lower="-1" upper="1" />
-  </joint>
-  <link name="lidar_with_mirror_mirror2_prismatic2_link">
-    <inertial>
-      <origin xyz="0 0 0" />
-      <mass value="0.01" />
-      <inertia ixx="0.1" ixy="0.0" ixz="0.0" iyy="0.1" iyz="0.0" izz="0.1" />
-    </inertial>
-  </link>
-  <xacro:include filename="$(find icart_mini_description)/urdf/sensors/hokuyo.urdf.xacro"/>
-  <xacro:sensor_hokuyo name="lidar_with_mirror_left" parent="lidar_with_mirror_mirror2_prismatic2_link">
-    <origin xyz="0 0 0" rpy="0 0 0"/>
-  </xacro:sensor_hokuyo>
+  </xacro:lidar_with_mirror>
   <transmission name="tran1">
     <type>transmission_interface/SimpleTransmission</type>
@@ -412,24 +289,4 @@
     </actuator>
   </transmission>
-  <transmission name="tran5">
-    <type>transmission_interface/SimpleTransmission</type>
-    <joint name="lidar_with_mirror_mirror1_roll_joint">
-      <hardwareInterface>hardware_interface/PositionJointInterface</hardwareInterface>
-    </joint>
-  <actuator name="lidar_with_mirror_mirror1_roll_motor">
-      <hardwareInterface>hardware_interface/PositionJointInterface</hardwareInterface>
-      <mechanicalReduction>1</mechanicalReduction>
-    </actuator>
-  </transmission>
-  <transmission name="tran6">
-    <type>transmission_interface/SimpleTransmission</type>
-    <joint name="lidar_with_mirror_mirror2_roll_joint">
-      <hardwareInterface>hardware_interface/PositionJointInterface</hardwareInterface>
-    </joint>
-  <actuator name="lidar_with_mirror_mirror2_roll_motor">
-      <hardwareInterface>hardware_interface/PositionJointInterface</hardwareInterface>
-      <mechanicalReduction>1</mechanicalReduction>
-    </actuator>
-  </transmission>
   <transmission name="tran7">
     <type>transmission_interface/SimpleTransmission</type>
@@ -462,63 +319,3 @@
     </actuator>
   </transmission>
-  <transmission name="tran10">
-    <type>transmission_interface/SimpleTransmission</type>
-    <joint name="lidar_with_mirror_mirror1_prismatic_joint">
-      <hardwareInterface>hardware_interface/PositionJointInterface</hardwareInterface>
-    </joint>
-    <actuator name="lidar_with_mirror_mirror1_prismatic_motor">
-      <hardwareInterface>hardware_interface/PositionJointInterface</hardwareInterface>
-      <mechanicalReduction>1</mechanicalReduction>
-    </actuator>
-  </transmission>
-  <transmission name="tran11">
-    <type>transmission_interface/SimpleTransmission</type>
-    <joint name="lidar_with_mirror_mirror2_prismatic_joint">
-      <hardwareInterface>hardware_interface/PositionJointInterface</hardwareInterface>
-    </joint>
-    <actuator name="lidar_with_mirror_mirror2_prismatic_motor">
-      <hardwareInterface>hardware_interface/PositionJointInterface</hardwareInterface>
-      <mechanicalReduction>1</mechanicalReduction>
-    </actuator>
-  </transmission>
-  <transmission name="tran12">
-    <type>transmission_interface/SimpleTransmission</type>
-    <joint name="lidar_with_mirror_mirror1_prismatic2_joint">
-      <hardwareInterface>hardware_interface/PositionJointInterface</hardwareInterface>
-    </joint>
-    <actuator name="lidar_with_mirror_mirror1_prismatic2_motor">
-      <hardwareInterface>hardware_interface/PositionJointInterface</hardwareInterface>
-      <mechanicalReduction>1</mechanicalReduction>
-    </actuator>
-  </transmission>
-  <transmission name="tran13">
-    <type>transmission_interface/SimpleTransmission</type>
-    <joint name="lidar_with_mirror_mirror2_prismatic2_joint">
-      <hardwareInterface>hardware_interface/PositionJointInterface</hardwareInterface>
-    </joint>
-    <actuator name="lidar_with_mirror_mirror2_prismatic2_motor">
-      <hardwareInterface>hardware_interface/PositionJointInterface</hardwareInterface>
-      <mechanicalReduction>1</mechanicalReduction>
-    </actuator>
-  </transmission>
-  <transmission name="tran14">
-    <type>transmission_interface/SimpleTransmission</type>
-    <joint name="lidar_with_mirror_mirror1_yaw_joint">
-      <hardwareInterface>hardware_interface/PositionJointInterface</hardwareInterface>
-    </joint>
-  <actuator name="lidar_with_mirror_mirror1_yaw_motor">
-      <hardwareInterface>hardware_interface/PositionJointInterface</hardwareInterface>
-      <mechanicalReduction>1</mechanicalReduction>
-    </actuator>
-  </transmission>
-  <transmission name="tran15">
-    <type>transmission_interface/SimpleTransmission</type>
-    <joint name="lidar_with_mirror_mirror2_yaw_joint">
-      <hardwareInterface>hardware_interface/PositionJointInterface</hardwareInterface>
-    </joint>
-  <actuator name="lidar_with_mirror_mirror2_yaw_motor">
-      <hardwareInterface>hardware_interface/PositionJointInterface</hardwareInterface>
-      <mechanicalReduction>1</mechanicalReduction>
-    </actuator>
-  </transmission>
 </robot>
