Commit message: add estimate_posture

File: lidar_with_mirror_description/urdf/orne_box_lidar_with_mirror.urdf.xacro (robot description, xacro)
@@ -202,5 +202,5 @@
     <parent link="lidar_with_mirror_prismatic_link"/>
     <child link="lidar_with_mirror_pitch_link"/>
-    <origin xyz="0 0 0" rpy="0 0 0"/>
+    <origin xyz="0 0 0" rpy="0 ${PI/9} 0"/>
     <axis xyz="0 1 0"/>
     <limit effort="100" velocity="100.0" lower="${-PI}" upper="${PI}" />
@@ -237,5 +237,5 @@
     <parent link="lidar_with_mirror_center_link"/>
     <child link="lidar_with_mirror_mirror1_roll_link"/>
-    <origin xyz="0 ${len} 0" rpy="0 0 0"/>
+    <origin xyz="0 ${len} 0" rpy="${-PI/2} 0 0"/>
     <axis xyz="-1 0 0"/>
     <limit effort="100" velocity="100.0" lower="${-PI}" upper="${PI}" />
@@ -255,5 +255,5 @@
     <parent link="lidar_with_mirror_center_link"/>
     <child link="lidar_with_mirror_mirror2_roll_link"/>
-    <origin xyz="0 ${-len} 0" rpy="0 0 0"/>
+    <origin xyz="0 ${-len} 0" rpy="${PI/2} 0 0"/>
     <axis xyz="1 0 0"/>
     <limit effort="100" velocity="100.0" lower="${-PI}" upper="${PI}" />

Commit message: add prismatic link

File: lidar_with_mirror_description/urdf/orne_box_lidar_with_mirror.urdf.xacro (robot description, xacro)
@@ -252,8 +252,22 @@
     <origin xyz="${front} 0 ${height}" rpy="0 0 0"/>
   </xacro:sensor_hokuyo>
+  <joint name="lidar_with_mirror_mirror1_prismatic_joint" type="prismatic">
+    <parent link="lidar_with_mirror_center_link"/>
+    <child link="lidar_with_mirror_mirror1_prismatic_link"/>
+    <origin xyz="0 ${len} 0" rpy="0 0 0"/>
+    <axis xyz="0 1 0"/>
+    <limit effort="100" velocity="100.0" lower="-1" upper="1" />
+  </joint>
+  <link name="lidar_with_mirror_mirror1_prismatic_link">
+    <inertial>
+      <origin xyz="0 0 0" />
+      <mass value="0.2" />
+      <inertia ixx="0.1" ixy="0.0" ixz="0.0" iyy="0.1" iyz="0.0" izz="0.1" />
+    </inertial>
+  </link>
   <joint name="lidar_with_mirror_mirror1_roll_joint" type="revolute">
-    <parent link="lidar_with_mirror_center_link"/>
+    <parent link="lidar_with_mirror_mirror1_prismatic_link"/>
     <child link="lidar_with_mirror_mirror1_roll_link"/>
-    <origin xyz="0 ${len} 0" rpy="${-PI/4} 0 0"/>
+    <origin xyz="0 0 0" rpy="${-PI/4} 0 0"/>
     <axis xyz="-1 0 0"/>
     <limit effort="100" velocity="100.0" lower="${-PI}" upper="${PI}" />
@@ -270,8 +284,22 @@
     <origin xyz="0 ${-len} 0" rpy="0 0 0"/>
   </xacro:sensor_hokuyo>
+  <joint name="lidar_with_mirror_mirror2_prismatic_joint" type="prismatic">
+    <parent link="lidar_with_mirror_center_link"/>
+    <child link="lidar_with_mirror_mirror2_prismatic_link"/>
+    <origin xyz="0 ${-len} 0" rpy="0 0 0"/>
+    <axis xyz="0 1 0"/>
+    <limit effort="100" velocity="100.0" lower="-1" upper="1" />
+  </joint>
+  <link name="lidar_with_mirror_mirror2_prismatic_link">
+    <inertial>
+      <origin xyz="0 0 0" />
+      <mass value="0.2" />
+      <inertia ixx="0.1" ixy="0.0" ixz="0.0" iyy="0.1" iyz="0.0" izz="0.1" />
+    </inertial>
+  </link>
   <joint name="lidar_with_mirror_mirror2_roll_joint" type="revolute">
-    <parent link="lidar_with_mirror_center_link"/>
+    <parent link="lidar_with_mirror_mirror2_prismatic_link"/>
     <child link="lidar_with_mirror_mirror2_roll_link"/>
-    <origin xyz="0 ${-len} 0" rpy="${PI/4} 0 0"/>
+    <origin xyz="0 0 0" rpy="${PI/4} 0 0"/>
     <axis xyz="1 0 0"/>
     <limit effort="100" velocity="100.0" lower="${-PI}" upper="${PI}" />
@@ -378,3 +406,23 @@
     </actuator>
   </transmission>
+  <transmission name="tran10">
+    <type>transmission_interface/SimpleTransmission</type>
+    <joint name="lidar_with_mirror_mirror1_prismatic_joint">
+      <hardwareInterface>hardware_interface/PositionJointInterface</hardwareInterface>
+    </joint>
+    <actuator name="lidar_with_mirror_mirror1_prismatic_motor">
+      <hardwareInterface>hardware_interface/PositionJointInterface</hardwareInterface>
+      <mechanicalReduction>1</mechanicalReduction>
+    </actuator>
+  </transmission>
+  <transmission name="tran11">
+    <type>transmission_interface/SimpleTransmission</type>
+    <joint name="lidar_with_mirror_mirror2_prismatic_joint">
+      <hardwareInterface>hardware_interface/PositionJointInterface</hardwareInterface>
+    </joint>
+    <actuator name="lidar_with_mirror_mirror2_prismatic_motor">
+      <hardwareInterface>hardware_interface/PositionJointInterface</hardwareInterface>
+      <mechanicalReduction>1</mechanicalReduction>
+    </actuator>
+  </transmission>
 </robot>

Commit message: control yaw angle

File: lidar_with_mirror_description/urdf/orne_box_lidar_with_mirror.urdf.xacro (robot description, xacro)
@@ -262,10 +262,24 @@
     <inertial>
       <origin xyz="0 0 0" />
-      <mass value="0.2" />
+      <mass value="0.01" />
+      <inertia ixx="0.1" ixy="0.0" ixz="0.0" iyy="0.1" iyz="0.0" izz="0.1" />
+    </inertial>
+  </link>
+  <joint name="lidar_with_mirror_mirror1_yaw_joint" type="revolute">
+    <parent link="lidar_with_mirror_mirror1_prismatic_link"/>
+    <child link="lidar_with_mirror_mirror1_yaw_link"/>
+    <origin xyz="0 0 0" rpy="0 0 0"/>
+    <axis xyz="0 0 1"/>
+    <limit effort="100" velocity="100.0" lower="${-PI}" upper="${PI}" />
+  </joint>
+  <link name="lidar_with_mirror_mirror1_yaw_link">
+    <inertial>
+      <origin xyz="0 0 0" />
+      <mass value="0.01" />
       <inertia ixx="0.1" ixy="0.0" ixz="0.0" iyy="0.1" iyz="0.0" izz="0.1" />
     </inertial>
   </link>
   <joint name="lidar_with_mirror_mirror1_roll_joint" type="revolute">
-    <parent link="lidar_with_mirror_mirror1_prismatic_link"/>
+    <parent link="lidar_with_mirror_mirror1_yaw_link"/>
     <child link="lidar_with_mirror_mirror1_roll_link"/>
     <origin xyz="0 0 0" rpy="${-PI/4} 0 0"/>
@@ -276,11 +290,25 @@
     <inertial>
       <origin xyz="0 0 0" />
-      <mass value="0.2" />
+      <mass value="0.01" />
+      <inertia ixx="0.1" ixy="0.0" ixz="0.0" iyy="0.1" iyz="0.0" izz="0.1" />
+    </inertial>
+  </link>
+  <joint name="lidar_with_mirror_mirror1_prismatic2_joint" type="prismatic">
+    <parent link="lidar_with_mirror_mirror1_roll_link"/>
+    <child link="lidar_with_mirror_mirror1_prismatic2_link"/>
+    <origin xyz="0 ${-len} 0" rpy="0 0 0"/>
+    <axis xyz="0 -1 0"/>
+    <limit effort="100" velocity="100.0" lower="-1" upper="1" />
+  </joint>
+  <link name="lidar_with_mirror_mirror1_prismatic2_link">
+    <inertial>
+      <origin xyz="0 0 0" />
+      <mass value="0.01" />
       <inertia ixx="0.1" ixy="0.0" ixz="0.0" iyy="0.1" iyz="0.0" izz="0.1" />
     </inertial>
   </link>
   <xacro:include filename="$(find icart_mini_description)/urdf/sensors/hokuyo.urdf.xacro"/>
-  <xacro:sensor_hokuyo name="lidar_with_mirror_left" parent="lidar_with_mirror_mirror1_roll_link">
-    <origin xyz="0 ${-len} 0" rpy="0 0 0"/>
+  <xacro:sensor_hokuyo name="lidar_with_mirror_left" parent="lidar_with_mirror_mirror1_prismatic2_link">
+    <origin xyz="0 0 0" rpy="0 0 0"/>
   </xacro:sensor_hokuyo>
   <joint name="lidar_with_mirror_mirror2_prismatic_joint" type="prismatic">
@@ -298,6 +326,20 @@
     </inertial>
   </link>
+  <joint name="lidar_with_mirror_mirror2_yaw_joint" type="revolute">
+    <parent link="lidar_with_mirror_mirror2_prismatic_link"/>
+    <child link="lidar_with_mirror_mirror2_yaw_link"/>
+    <origin xyz="0 0 0" rpy="0 0 0"/>
+    <axis xyz="0 0 1"/>
+    <limit effort="100" velocity="100.0" lower="${-PI}" upper="${PI}" />
+  </joint>
+  <link name="lidar_with_mirror_mirror2_yaw_link">
+    <inertial>
+      <origin xyz="0 0 0" />
+      <mass value="0.01" />
+      <inertia ixx="0.1" ixy="0.0" ixz="0.0" iyy="0.1" iyz="0.0" izz="0.1" />
+    </inertial>
+  </link>
   <joint name="lidar_with_mirror_mirror2_roll_joint" type="revolute">
-    <parent link="lidar_with_mirror_mirror2_prismatic_link"/>
+    <parent link="lidar_with_mirror_mirror2_yaw_link"/>
     <child link="lidar_with_mirror_mirror2_roll_link"/>
     <origin xyz="0 0 0" rpy="${PI/4} 0 0"/>
@@ -312,7 +354,21 @@
     </inertial>
   </link>
+  <joint name="lidar_with_mirror_mirror2_prismatic2_joint" type="prismatic">
+    <parent link="lidar_with_mirror_mirror2_roll_link"/>
+    <child link="lidar_with_mirror_mirror2_prismatic2_link"/>
+    <origin xyz="0 ${len} 0" rpy="0 0 0"/>
+    <axis xyz="0 1 0"/>
+    <limit effort="100" velocity="100.0" lower="-1" upper="1" />
+  </joint>
+  <link name="lidar_with_mirror_mirror2_prismatic2_link">
+    <inertial>
+      <origin xyz="0 0 0" />
+      <mass value="0.01" />
+      <inertia ixx="0.1" ixy="0.0" ixz="0.0" iyy="0.1" iyz="0.0" izz="0.1" />
+    </inertial>
+  </link>
   <xacro:include filename="$(find icart_mini_description)/urdf/sensors/hokuyo.urdf.xacro"/>
-  <xacro:sensor_hokuyo name="lidar_with_mirror_right" parent="lidar_with_mirror_mirror2_roll_link">
-    <origin xyz="0 ${len} 0" rpy="0 0 0"/>
+  <xacro:sensor_hokuyo name="lidar_with_mirror_right" parent="lidar_with_mirror_mirror2_prismatic2_link">
+    <origin xyz="0 0 0" rpy="0 0 0"/>
   </xacro:sensor_hokuyo>
   <transmission name="tran1">
@@ -426,3 +482,43 @@
     </actuator>
   </transmission>
+  <transmission name="tran12">
+    <type>transmission_interface/SimpleTransmission</type>
+    <joint name="lidar_with_mirror_mirror1_prismatic2_joint">
+      <hardwareInterface>hardware_interface/PositionJointInterface</hardwareInterface>
+    </joint>
+    <actuator name="lidar_with_mirror_mirror1_prismatic2_motor">
+      <hardwareInterface>hardware_interface/PositionJointInterface</hardwareInterface>
+      <mechanicalReduction>1</mechanicalReduction>
+    </actuator>
+  </transmission>
+  <transmission name="tran13">
+    <type>transmission_interface/SimpleTransmission</type>
+    <joint name="lidar_with_mirror_mirror2_prismatic2_joint">
+      <hardwareInterface>hardware_interface/PositionJointInterface</hardwareInterface>
+    </joint>
+    <actuator name="lidar_with_mirror_mirror2_prismatic2_motor">
+      <hardwareInterface>hardware_interface/PositionJointInterface</hardwareInterface>
+      <mechanicalReduction>1</mechanicalReduction>
+    </actuator>
+  </transmission>
+  <transmission name="tran14">
+    <type>transmission_interface/SimpleTransmission</type>
+    <joint name="lidar_with_mirror_mirror1_yaw_joint">
+      <hardwareInterface>hardware_interface/PositionJointInterface</hardwareInterface>
+    </joint>
+  <actuator name="lidar_with_mirror_mirror1_yaw_motor">
+      <hardwareInterface>hardware_interface/PositionJointInterface</hardwareInterface>
+      <mechanicalReduction>1</mechanicalReduction>
+    </actuator>
+  </transmission>
+  <transmission name="tran15">
+    <type>transmission_interface/SimpleTransmission</type>
+    <joint name="lidar_with_mirror_mirror2_yaw_joint">
+      <hardwareInterface>hardware_interface/PositionJointInterface</hardwareInterface>
+    </joint>
+  <actuator name="lidar_with_mirror_mirror2_yaw_motor">
+      <hardwareInterface>hardware_interface/PositionJointInterface</hardwareInterface>
+      <mechanicalReduction>1</mechanicalReduction>
+    </actuator>
+  </transmission>
 </robot>

Commit message: calculate pose

File: lidar_with_mirror_description/urdf/orne_box_lidar_with_mirror.urdf.xacro (robot description, xacro)
@@ -213,5 +213,5 @@
     <inertial>
       <origin xyz="0 0 0" />
-      <mass value="0.2" />
+      <mass value="0.01" />
       <inertia ixx="0.1" ixy="0.0" ixz="0.0" iyy="0.1" iyz="0.0" izz="0.1" />
     </inertial>
@@ -227,5 +227,5 @@
     <inertial>
       <origin xyz="0 0 0" />
-      <mass value="0.2" />
+      <mass value="0.01" />
       <inertia ixx="0.1" ixy="0.0" ixz="0.0" iyy="0.1" iyz="0.0" izz="0.1" />
     </inertial>
@@ -241,5 +241,5 @@
     <inertial>
       <origin xyz="0 0 0" />
-      <mass value="0.2" />
+      <mass value="0.01" />
       <inertia ixx="0.1" ixy="0.0" ixz="0.0" iyy="0.1" iyz="0.0" izz="0.1" />
     </inertial>
@@ -316,5 +316,5 @@
     <child link="lidar_with_mirror_mirror2_prismatic_link"/>
     <origin xyz="0 ${-len} 0" rpy="0 0 0"/>
-    <axis xyz="0 1 0"/>
+    <axis xyz="0 -1 0"/>
     <limit effort="100" velocity="100.0" lower="-1" upper="1" />
   </joint>
@@ -322,5 +322,5 @@
     <inertial>
       <origin xyz="0 0 0" />
-      <mass value="0.2" />
+      <mass value="0.01" />
       <inertia ixx="0.1" ixy="0.0" ixz="0.0" iyy="0.1" iyz="0.0" izz="0.1" />
     </inertial>
@@ -350,5 +350,5 @@
     <inertial>
       <origin xyz="0 0 0" />
-      <mass value="0.2" />
+      <mass value="0.01" />
       <inertia ixx="0.1" ixy="0.0" ixz="0.0" iyy="0.1" iyz="0.0" izz="0.1" />
     </inertial>

Commit message: description

File: lidar_with_mirror_description/urdf/orne_box_lidar_with_mirror.urdf.xacro (robot description, xacro)
@@ -1,204 +1,10 @@
 <?xml version="1.0" ?>
 <robot name="orne_box" xmlns:xacro="http://www.ros.org/wiki/xacro">
+  <xacro:arg name="ignition_gazebo" default="false"/>
   <xacro:property name="PI" value="3.1415926535897931"/>
-  <xacro:include filename="$(find icart_mini_description)/urdf/materials.xacro" />
+  <xacro:include filename="$(find orne_box_description)/urdf/orne_box.urdf.xacro" />
   <xacro:include filename="$(find lidar_with_mirror_description)/urdf/orne_box_lidar_with_mirror.gazebo.xacro"/>
-  <link name="base_link">
-<!--
-    <visual>
-      <origin xyz="0 0 -0.154" rpy="0 0 0"/>
-      <geometry>
-        <mesh filename="package://orne_box_description/meshes/bases/orne_box_base.stl" scale="1 1 1"/>
-      </geometry>
-      <material name="orange"/>
-    </visual>
--->
-    <visual>
-      <origin xyz="0.090 0 0.1715" rpy="0 0 0"/>
-      <geometry>
-        <box size="0.400 0.404 0.202"/>
-      </geometry>
-      <material name="orange"/>
-    </visual>
-    <visual>
-      <origin xyz="0.36125 0 0.2625" rpy="0 0 0"/>
-      <geometry>
-        <box size="0.1425 0.404 0.020"/>
-      </geometry>
-      <material name="orange"/>
-    </visual>
-    <visual>
-      <origin xyz="0.35625 0 0.156" rpy="0 0 0"/>
-      <geometry>
-        <box size="0.1325 0.404 0.020"/>
-      </geometry>
-      <material name="orange"/>
-    </visual>
-    <visual>
-      <origin xyz="-0.120 0 0.4815" rpy="0 0 0"/>
-      <geometry>
-        <box size="0.020 0.404 0.822"/>
-      </geometry>
-      <material name="orange"/>
-    </visual>
-<!--
-    <collision>
-      <origin xyz="0.090 0 0.1715" rpy="0 0 0"/>
-      <geometry>
-        <box size="0.400 0.404 0.202"/>
-      </geometry>
-    </collision>
-    <collision>
-      <origin xyz="0.36125 0 0.2625" rpy="0 0 0"/>
-      <geometry>
-        <box size="0.1425 0.404 0.020"/>
-      </geometry>
-    </collision>
-    <collision>
-      <origin xyz="0.35625 0 0.156" rpy="0 0 0"/>
-      <geometry>
-        <box size="0.1325 0.404 0.020"/>
-      </geometry>
-    </collision>
-    <collision>
-      <origin xyz="-0.120 0 0.4815" rpy="0 0 0"/>
-      <geometry>
-        <box size="0.020 0.404 0.822"/>
-      </geometry>
-    </collision>
--->
-    <inertial>
-      <origin xyz="0.090 0 0.1715" rpy="0 0 0"/>
-      <mass value="25.0"/>
-      <inertia ixx="1.0" ixy="0.0" ixz="0.0" iyy="1.0" iyz="0.0" izz="1.0" />
-    </inertial>
-  </link>
-  <joint name="wheel_hinge" type="revolute">
-    <parent link="base_link"/>
-    <child link="wheel_link"/>
-    <origin xyz="0.0 0.0 0.152" rpy="0 0 0"/>
-    <axis xyz="1 0 0"/>
-    <limit effort="100" velocity="100.0"  lower="-5000" upper="5000" />
-  </joint>
-  <link name="wheel_link">
-    <inertial>
-      <origin xyz="0 0 0" />
-      <mass value="0.2" />
-      <inertia ixx="0.1" ixy="0.0" ixz="0.0" iyy="0.1" iyz="0.0" izz="0.1" />
-    </inertial>
-  </link>
-  <joint name="left_wheel_hinge" type="revolute">
-    <parent link="wheel_link"/>
-    <child link="wheel_left_link"/>
-    <origin xyz="0.0 0.23075 0.0" rpy="${-PI/2} 0 0"/>
-    <axis xyz="0 0 1"/>
-    <limit effort="100" velocity="100.0"  lower="-5000" upper="5000" />
-  </joint>
-  <link name="wheel_left_link">
-    <visual>
-      <origin xyz="0 0 0" rpy="0 0 0"/>
-      <geometry>
-        <mesh filename="package://orne_box_description/meshes/wheels/tire.stl" scale="1 1 1"/>
-      </geometry>
-<!--
-      <origin xyz="0 0 0" rpy="0 0 0"/>
-      <geometry>
-        <cylinder length="0.045" radius="0.152"/>
-      </geometry>
--->
-      <material name="white"/>
-    </visual>
-    <collision>
-      <origin xyz="0 0 0" rpy="0 0 0"/>
-      <geometry>
-        <cylinder length="0.045" radius="0.152"/>
-      </geometry>
-    </collision>
-    <inertial>
-      <origin xyz="0 0 0" />
-      <mass value="0.2" />
-      <inertia ixx="0.1" ixy="0.0" ixz="0.0" iyy="0.1" iyz="0.0" izz="0.1" />
-    </inertial>
-  </link>
-  <joint name="right_wheel_hinge" type="revolute">
-    <parent link="wheel_link"/>
-    <child link="wheel_right_link"/>
-    <origin xyz="0.0 -0.23075 0.0" rpy="${-PI/2} 0 0"/>
-    <axis xyz="0 0 1"/>
-    <limit effort="100" velocity="100.0"  lower="-5000" upper="5000" />
-  </joint>
-  <link name="wheel_right_link">
-    <visual>
-      <origin xyz="0 0 0" rpy="0 0 0"/>
-      <geometry>
-        <mesh filename="package://orne_box_description/meshes/wheels/tire.stl" scale="1 1 1"/>
-      </geometry>
-<!--
-      <origin xyz="0 0 0" rpy="0 0 0"/>
-      <geometry>
-        <cylinder length="0.045" radius="0.152"/>
-      </geometry>
--->
-      <material name="white"/>
-    </visual>
-    <collision>
-      <origin xyz="0 0 0" rpy="0 0 0"/>
-      <geometry>
-        <cylinder length="0.045" radius="0.152"/>
-      </geometry>
-    </collision>
-    <inertial>
-      <origin xyz="0 0 0" />
-      <mass value="0.2" />
-      <inertia ixx="0.1" ixy="0.0" ixz="0.0" iyy="0.1" iyz="0.0" izz="0.1" />
-    </inertial>
-  </link>
-  <joint name="caster_front_joint" type="prismatic">
-    <parent link="base_link"/>
-    <child link="caster_front_link"/>
-    <origin xyz="0.362 0 0.050" rpy="0 0 0"/>
-    <axis xyz="0 0 1"/>
-    <limit effort="100" velocity="100.0" lower="-1" upper="1" />
-  </joint>
-  <link name="caster_front_link">
-    <visual>
-      <origin xyz="0 0.150 0" rpy="${PI/2} 0 0"/>
-      <geometry>
-        <cylinder length="0.025" radius="0.050"/>
-      </geometry>
-      <material name="red"/>
-    </visual>
-    <visual>
-      <origin xyz="0 -0.150 0" rpy="${PI/2} 0 0"/>
-      <geometry>
-        <cylinder length="0.025" radius="0.050"/>
-      </geometry>
-      <material name="red"/>
-    </visual>
-    <collision>
-      <origin xyz="0 0.150 0" rpy="${PI/2} 0 0"/>
-      <geometry>
-        <cylinder length="0.025" radius="0.050"/>
-      </geometry>
-    </collision>
-    <collision>
-      <origin xyz="0 -0.150 0" rpy="${PI/2} 0 0"/>
-      <geometry>
-        <cylinder length="0.025" radius="0.050"/>
-      </geometry>
-    </collision>
-    <inertial>
-      <origin xyz="0 0 0" />
-      <mass value="0.2" />
-      <inertia ixx="0.1" ixy="0.0" ixz="0.0" iyy="0.1" iyz="0.0" izz="0.1" />
-    </inertial>
-  </link>
-  <xacro:include filename="$(find icart_mini_description)/urdf/sensors/imu.urdf.xacro"/>
-  <!-- Setting for imu -->
-  <xacro:sensor_imu name="imu" parent="base_link" size="0.05 0.05 0.05">
-    <origin xyz="0.3 0 0.2445" rpy="0 0 ${-PI/2}"/>
-  </xacro:sensor_imu>
-  <xacro:include filename="$(find icart_mini_description)/urdf/sensors/hokuyo.urdf.xacro"/>
-  <xacro:sensor_hokuyo name="hokuyo" parent="base_link">
+  <xacro:include filename="$(find orne_box_description)/urdf/sensors/hokuyo.urdf.xacro"/>
+  <xacro:sensor_hokuyo name="hokuyo_with_mirror" parent="base_link" size="0.05 0.05 0.05">
     <origin xyz="0.374295 0 0.2185" rpy="${-PI} 0 0"/>
   </xacro:sensor_hokuyo>
@@ -245,9 +51,8 @@
     </inertial>
   </link>
-  <xacro:property name="len" value="0.1" />
+  <xacro:property name="len0" value="0.1" />
   <xacro:property name="front" value="0" />
   <xacro:property name="height" value="0" />
-  <xacro:include filename="$(find icart_mini_description)/urdf/sensors/hokuyo.urdf.xacro"/>
-  <xacro:sensor_hokuyo name="lidar_with_mirror_center" parent="lidar_with_mirror_roll_link">
+  <xacro:sensor_hokuyo name="lidar_with_mirror_center" parent="lidar_with_mirror_roll_link" size="0.05 0.05 0.05">
     <origin xyz="${front} 0 ${height}" rpy="0 0 0"/>
   </xacro:sensor_hokuyo>
@@ -255,5 +60,5 @@
     <parent link="lidar_with_mirror_center_link"/>
     <child link="lidar_with_mirror_mirror1_roll_link"/>
-    <origin xyz="0 ${len} 0" rpy="${-PI/4} 0 0"/>
+    <origin xyz="0 ${len0} 0" rpy="${-PI/4} 0 0"/>
     <axis xyz="-1 0 0"/>
     <limit effort="100" velocity="100.0" lower="${-PI}" upper="${PI}" />
@@ -266,12 +71,11 @@
     </inertial>
   </link>
-  <xacro:include filename="$(find icart_mini_description)/urdf/sensors/hokuyo.urdf.xacro"/>
-  <xacro:sensor_hokuyo name="lidar_with_mirror_left" parent="lidar_with_mirror_mirror1_roll_link">
-    <origin xyz="0 ${-len} 0" rpy="0 0 0"/>
+  <xacro:sensor_hokuyo name="lidar_with_mirror_left" parent="lidar_with_mirror_mirror1_roll_link"  size="0.05 0.05 0.05">
+    <origin xyz="0 ${-len0} 0" rpy="0 0 0"/>
   </xacro:sensor_hokuyo>
   <joint name="lidar_with_mirror_mirror2_roll_joint" type="revolute">
     <parent link="lidar_with_mirror_center_link"/>
     <child link="lidar_with_mirror_mirror2_roll_link"/>
-    <origin xyz="0 ${-len} 0" rpy="${PI/4} 0 0"/>
+    <origin xyz="0 ${-len0} 0" rpy="${PI/4} 0 0"/>
     <axis xyz="1 0 0"/>
     <limit effort="100" velocity="100.0" lower="${-PI}" upper="${PI}" />
@@ -284,7 +88,6 @@
     </inertial>
   </link>
-  <xacro:include filename="$(find icart_mini_description)/urdf/sensors/hokuyo.urdf.xacro"/>
-  <xacro:sensor_hokuyo name="lidar_with_mirror_right" parent="lidar_with_mirror_mirror2_roll_link">
-    <origin xyz="0 ${len} 0" rpy="0 0 0"/>
+  <xacro:sensor_hokuyo name="lidar_with_mirror_right" parent="lidar_with_mirror_mirror2_roll_link"  size="0.05 0.05 0.05">
+    <origin xyz="0 ${len0} 0" rpy="0 0 0"/>
   </xacro:sensor_hokuyo>
   <transmission name="tran1">
@@ -358,23 +161,3 @@
     </actuator>
   </transmission>
-  <transmission name="tran8">
-    <type>transmission_interface/SimpleTransmission</type>
-    <joint name="caster_front_joint">
-      <hardwareInterface>hardware_interface/PositionJointInterface</hardwareInterface>
-    </joint>
-  <actuator name="caster_front_motor">
-      <hardwareInterface>hardware_interface/PositionJointInterface</hardwareInterface>
-      <mechanicalReduction>1</mechanicalReduction>
-    </actuator>
-  </transmission>
-  <transmission name="tran9">
-    <type>transmission_interface/SimpleTransmission</type>
-    <joint name="wheel_hinge">
-      <hardwareInterface>hardware_interface/PositionJointInterface</hardwareInterface>
-    </joint>
-  <actuator name="wheel_hinge_motor">
-      <hardwareInterface>hardware_interface/PositionJointInterface</hardwareInterface>
-      <mechanicalReduction>1</mechanicalReduction>
-    </actuator>
-  </transmission>
 </robot>
