Commit message: rename

File: lidar_with_mirror_description/urdf/check_lidar_with_mirror.urdf.xacro (robot description, xacro)
@@ -4,5 +4,5 @@
   <xacro:include filename="$(find lidar_with_mirror_description)/urdf/sensor/lidar_with_mirror.urdf.xacro" />
   <link name="base_link"/>
-  <xacro:lidar_with_mirror name="lidar_with_mirror" parent="base_link" left_roll_rad="0.769999299112962" left_pitch_rad="-0.05" left_distance_m="0.073124500184212" right_roll_rad="0.787426157712581" right_pitch_rad="-0.05" right_distance_m="0.072588298861567">
+  <xacro:lidar_with_mirror name="lidar_with_mirror" parent="base_link" right_roll_rad="0.769999299112962" left_pitch_rad="-0.05" right_distance_m="0.073124500184212" left_roll_rad="0.787426157712581" right_pitch_rad="-0.05" left_distance_m="0.072588298861567">
     <origin xyz="0 0 0" rpy="0 0 0"/>
   </xacro:lidar_with_mirror>

File: lidar_with_mirror_description/urdf/orne_box_lidar_with_mirror.urdf.xacro (robot description, xacro)
@@ -195,4 +195,5 @@
     <origin xyz="0.374295 0 0.2185" rpy="${-PI} 0 0"/>
   </xacro:sensor_hokuyo>
+  <!-- Setting for Lidar with mirror -->
   <joint name="lidar_with_mirror_prismatic_joint" type="prismatic">
     <parent link="base_link"/>
@@ -238,5 +239,5 @@
   </link>
   <xacro:include filename="$(find lidar_with_mirror_description)/urdf/sensor/lidar_with_mirror.urdf.xacro" />
-  <xacro:lidar_with_mirror name="lidar_with_mirror" parent="lidar_with_mirror_roll_link" left_roll_rad="${radians(70)}" left_pitch_rad="0.0" left_distance_m="0.21" right_roll_rad="${radians(70)}" right_pitch_rad="0.0" right_distance_m="0.21">
+  <xacro:lidar_with_mirror name="lidar_with_mirror" parent="lidar_with_mirror_roll_link" right_roll_rad="${radians(70)}" left_pitch_rad="0.0" right_distance_m="0.21" left_roll_rad="${radians(70)}" right_pitch_rad="0.0" left_distance_m="0.21">
     <origin xyz="0 0 0" rpy="0 0 0"/>
   </xacro:lidar_with_mirror>

File: lidar_with_mirror_description/urdf/sensor/lidar_with_mirror.urdf.xacro (robot description, xacro)
@@ -2,5 +2,5 @@
 <robot name="lidar_with_mirror" xmlns:xacro="http://www.ros.org/wiki/xacro">
   <xacro:property name="PI" value="3.1415926535897931"/>
-  <xacro:macro name="lidar_with_mirror" params="name parent *origin left_roll_rad left_pitch_rad left_distance_m right_roll_rad right_pitch_rad right_distance_m">
+  <xacro:macro name="lidar_with_mirror" params="name parent *origin right_roll_rad left_pitch_rad right_distance_m left_roll_rad right_pitch_rad left_distance_m">
     <joint name="${name}_joint" type="fixed">
       <axis xyz="0 0 1"/>
@@ -18,207 +18,206 @@
     <xacro:include filename="$(find icart_mini_description)/urdf/sensors/hokuyo.urdf.xacro"/>
     <xacro:sensor_hokuyo name="${name}_center" parent="${name}_link">
-      <origin xyz="0 0 0" rpy="${PI} 0 0"/>
+      <origin xyz="0 0 0" rpy="0 0 0"/>
     </xacro:sensor_hokuyo>
-    <joint name="${name}_mirror1_prismatic_joint" type="prismatic">
+    <joint name="${name}_left_prismatic_joint" type="prismatic">
       <parent link="${name}_center_link"/>
-      <child link="${name}_mirror1_prismatic_link"/>
+      <child link="${name}_left_prismatic_link"/>
+      <origin xyz="0 ${left_distance_m} 0" rpy="0 0 0"/>
+      <axis xyz="0 1 0"/>
+      <limit effort="100" velocity="100.0" lower="-1" upper="1" />
+    </joint>
+    <link name="${name}_left_prismatic_link">
+      <inertial>
+        <origin xyz="0 0 0" />
+        <mass value="0.01" />
+        <inertia ixx="0.1" ixy="0.0" ixz="0.0" iyy="0.1" iyz="0.0" izz="0.1" />
+      </inertial>
+    </link>
+    <joint name="${name}_left_pitch_joint" type="revolute">
+      <parent link="${name}_left_prismatic_link"/>
+      <child link="${name}_left_yaw_link"/>
+      <origin xyz="0 0 0" rpy="0 ${right_pitch_rad} 0"/>
+      <axis xyz="0 1 0"/>
+      <limit effort="100" velocity="100.0" lower="${-PI}" upper="${PI}" />
+    </joint>
+    <link name="${name}_left_yaw_link">
+      <inertial>
+        <origin xyz="0 0 0" />
+        <mass value="0.01" />
+        <inertia ixx="0.1" ixy="0.0" ixz="0.0" iyy="0.1" iyz="0.0" izz="0.1" />
+      </inertial>
+    </link>
+    <joint name="${name}_left_roll_joint" type="revolute">
+      <parent link="${name}_left_yaw_link"/>
+      <child link="${name}_left_roll_link"/>
+      <origin xyz="0 0 0" rpy="${left_roll_rad} 0 0"/>
+      <axis xyz="1 0 0"/>
+      <limit effort="100" velocity="100.0" lower="${-PI}" upper="${PI}" />
+    </joint>
+    <link name="${name}_left_roll_link">
+      <inertial>
+        <origin xyz="0 0 0" />
+        <mass value="0.01" />
+        <inertia ixx="0.1" ixy="0.0" ixz="0.0" iyy="0.1" iyz="0.0" izz="0.1" />
+      </inertial>
+    </link>
+    <joint name="${name}_left_prismatic2_joint" type="prismatic">
+      <parent link="${name}_left_roll_link"/>
+      <child link="${name}_left_prismatic2_link"/>
+      <origin xyz="0 -${left_distance_m} 0" rpy="0 0 0"/>
+      <axis xyz="0 -1 0"/>
+      <limit effort="100" velocity="100.0" lower="-1" upper="1" />
+    </joint>
+    <link name="${name}_left_prismatic2_link">
+      <inertial>
+        <origin xyz="0 0 0" />
+        <mass value="0.01" />
+        <inertia ixx="0.1" ixy="0.0" ixz="0.0" iyy="0.1" iyz="0.0" izz="0.1" />
+      </inertial>
+    </link>
+    <xacro:include filename="$(find icart_mini_description)/urdf/sensors/hokuyo.urdf.xacro"/>
+    <xacro:sensor_hokuyo name="${name}_left" parent="${name}_left_prismatic2_link">
+      <origin xyz="0 0 0" rpy="0 0 0"/>
+    </xacro:sensor_hokuyo>
+    <joint name="${name}_right_prismatic_joint" type="prismatic">
+      <parent link="${name}_center_link"/>
+      <child link="${name}_right_prismatic_link"/>
+      <origin xyz="0 ${-right_distance_m} 0" rpy="0 0 0"/>
+      <axis xyz="0 -1 0"/>
+      <limit effort="100" velocity="100.0" lower="-1" upper="1" />
+    </joint>
+    <link name="${name}_right_prismatic_link">
+      <inertial>
+        <origin xyz="0 0 0" />
+        <mass value="0.01" />
+        <inertia ixx="0.1" ixy="0.0" ixz="0.0" iyy="0.1" iyz="0.0" izz="0.1" />
+      </inertial>
+    </link>
+    <joint name="${name}_right_pitch_joint" type="revolute">
+      <parent link="${name}_right_prismatic_link"/>
+      <child link="${name}_right_yaw_link"/>
+      <origin xyz="0 0 0" rpy="0 ${left_pitch_rad} 0"/>
+      <axis xyz="0 1 0"/>
+      <limit effort="100" velocity="100.0" lower="${-PI}" upper="${PI}" />
+    </joint>
+    <link name="${name}_right_yaw_link">
+      <inertial>
+        <origin xyz="0 0 0" />
+        <mass value="0.01" />
+        <inertia ixx="0.1" ixy="0.0" ixz="0.0" iyy="0.1" iyz="0.0" izz="0.1" />
+      </inertial>
+    </link>
+    <joint name="${name}_right_roll_joint" type="revolute">
+      <parent link="${name}_right_yaw_link"/>
+      <child link="${name}_right_roll_link"/>
+      <origin xyz="0 0 0" rpy="-${right_roll_rad} 0 0"/>
+      <axis xyz="-1 0 0"/>
+      <limit effort="100" velocity="100.0" lower="${-PI}" upper="${PI}" />
+    </joint>
+    <link name="${name}_right_roll_link">
+      <inertial>
+        <origin xyz="0 0 0" />
+        <mass value="0.01" />
+        <inertia ixx="0.1" ixy="0.0" ixz="0.0" iyy="0.1" iyz="0.0" izz="0.1" />
+      </inertial>
+    </link>
+    <joint name="${name}_right_prismatic2_joint" type="prismatic">
+      <parent link="${name}_right_roll_link"/>
+      <child link="${name}_right_prismatic2_link"/>
       <origin xyz="0 ${right_distance_m} 0" rpy="0 0 0"/>
       <axis xyz="0 1 0"/>
       <limit effort="100" velocity="100.0" lower="-1" upper="1" />
     </joint>
-  <link name="${name}_mirror1_prismatic_link">
-    <inertial>
-      <origin xyz="0 0 0" />
-      <mass value="0.01" />
-      <inertia ixx="0.1" ixy="0.0" ixz="0.0" iyy="0.1" iyz="0.0" izz="0.1" />
-    </inertial>
-  </link>
-  <joint name="${name}_mirror1_pitch_joint" type="revolute">
-    <parent link="${name}_mirror1_prismatic_link"/>
-    <child link="${name}_mirror1_yaw_link"/>
-    <origin xyz="0 0 0" rpy="0 ${right_pitch_rad} 0"/>
-    <axis xyz="0 1 0"/>
-    <limit effort="100" velocity="100.0" lower="${-PI}" upper="${PI}" />
-  </joint>
-  <link name="${name}_mirror1_yaw_link">
-    <inertial>
-      <origin xyz="0 0 0" />
-      <mass value="0.01" />
-      <inertia ixx="0.1" ixy="0.0" ixz="0.0" iyy="0.1" iyz="0.0" izz="0.1" />
-    </inertial>
-  </link>
-  <joint name="${name}_mirror1_roll_joint" type="revolute">
-    <parent link="${name}_mirror1_yaw_link"/>
-    <child link="${name}_mirror1_roll_link"/>
-    <origin xyz="0 0 0" rpy="${right_roll_rad} 0 0"/>
-    <axis xyz="1 0 0"/>
-    <limit effort="100" velocity="100.0" lower="${-PI}" upper="${PI}" />
-  </joint>
-  <link name="${name}_mirror1_roll_link">
-    <inertial>
-      <origin xyz="0 0 0" />
-      <mass value="0.01" />
-      <inertia ixx="0.1" ixy="0.0" ixz="0.0" iyy="0.1" iyz="0.0" izz="0.1" />
-    </inertial>
-  </link>
-  <joint name="${name}_mirror1_prismatic2_joint" type="prismatic">
-    <parent link="${name}_mirror1_roll_link"/>
-    <child link="${name}_mirror1_prismatic2_link"/>
-    <origin xyz="0 -${right_distance_m} 0" rpy="0 0 0"/>
-    <axis xyz="0 -1 0"/>
-    <limit effort="100" velocity="100.0" lower="-1" upper="1" />
-  </joint>
-  <link name="${name}_mirror1_prismatic2_link">
-    <inertial>
-      <origin xyz="0 0 0" />
-      <mass value="0.01" />
-      <inertia ixx="0.1" ixy="0.0" ixz="0.0" iyy="0.1" iyz="0.0" izz="0.1" />
-    </inertial>
-  </link>
-  <xacro:include filename="$(find icart_mini_description)/urdf/sensors/hokuyo.urdf.xacro"/>
-  <xacro:sensor_hokuyo name="${name}_right" parent="${name}_mirror1_prismatic2_link">
-    <origin xyz="0 0 0" rpy="0 0 0"/>
-  </xacro:sensor_hokuyo>
-  <joint name="${name}_mirror2_prismatic_joint" type="prismatic">
-    <parent link="${name}_center_link"/>
-    <child link="${name}_mirror2_prismatic_link"/>
-    <origin xyz="0 ${-left_distance_m} 0" rpy="0 0 0"/>
-    <axis xyz="0 -1 0"/>
-    <limit effort="100" velocity="100.0" lower="-1" upper="1" />
-  </joint>
-  <link name="${name}_mirror2_prismatic_link">
-    <inertial>
-      <origin xyz="0 0 0" />
-      <mass value="0.01" />
-      <inertia ixx="0.1" ixy="0.0" ixz="0.0" iyy="0.1" iyz="0.0" izz="0.1" />
-    </inertial>
-  </link>
-  <joint name="${name}_mirror2_pitch_joint" type="revolute">
-    <parent link="${name}_mirror2_prismatic_link"/>
-    <child link="${name}_mirror2_yaw_link"/>
-    <origin xyz="0 0 0" rpy="0 ${left_pitch_rad} 0"/>
-    <axis xyz="0 1 0"/>
-    <limit effort="100" velocity="100.0" lower="${-PI}" upper="${PI}" />
-  </joint>
-  <link name="${name}_mirror2_yaw_link">
-    <inertial>
-      <origin xyz="0 0 0" />
-      <mass value="0.01" />
-      <inertia ixx="0.1" ixy="0.0" ixz="0.0" iyy="0.1" iyz="0.0" izz="0.1" />
-    </inertial>
-  </link>
-  <joint name="${name}_mirror2_roll_joint" type="revolute">
-    <parent link="${name}_mirror2_yaw_link"/>
-    <child link="${name}_mirror2_roll_link"/>
-    <origin xyz="0 0 0" rpy="-${left_roll_rad} 0 0"/>
-    <axis xyz="-1 0 0"/>
-    <limit effort="100" velocity="100.0" lower="${-PI}" upper="${PI}" />
-  </joint>
-  <link name="${name}_mirror2_roll_link">
-    <inertial>
-      <origin xyz="0 0 0" />
-      <mass value="0.01" />
-      <inertia ixx="0.1" ixy="0.0" ixz="0.0" iyy="0.1" iyz="0.0" izz="0.1" />
-    </inertial>
-  </link>
-  <joint name="${name}_mirror2_prismatic2_joint" type="prismatic">
-    <parent link="${name}_mirror2_roll_link"/>
-    <child link="${name}_mirror2_prismatic2_link"/>
-    <origin xyz="0 ${left_distance_m} 0" rpy="0 0 0"/>
-    <axis xyz="0 1 0"/>
-    <limit effort="100" velocity="100.0" lower="-1" upper="1" />
-  </joint>
-  <link name="${name}_mirror2_prismatic2_link">
-    <inertial>
-      <origin xyz="0 0 0" />
-      <mass value="0.01" />
-      <inertia ixx="0.1" ixy="0.0" ixz="0.0" iyy="0.1" iyz="0.0" izz="0.1" />
-    </inertial>
-  </link>
-  <xacro:include filename="$(find icart_mini_description)/urdf/sensors/hokuyo.urdf.xacro"/>
-  <xacro:sensor_hokuyo name="${name}_left" parent="${name}_mirror2_prismatic2_link">
-    <origin xyz="0 0 0" rpy="0 0 0"/>
-  </xacro:sensor_hokuyo>
-  <transmission name="tran5">
-    <type>transmission_interface/SimpleTransmission</type>
-    <joint name="${name}_mirror1_roll_joint">
-      <hardwareInterface>hardware_interface/PositionJointInterface</hardwareInterface>
-    </joint>
-  <actuator name="${name}_mirror1_roll_motor">
-      <hardwareInterface>hardware_interface/PositionJointInterface</hardwareInterface>
-      <mechanicalReduction>1</mechanicalReduction>
-    </actuator>
-  </transmission>
-  <transmission name="tran6">
-    <type>transmission_interface/SimpleTransmission</type>
-    <joint name="${name}_mirror2_roll_joint">
-      <hardwareInterface>hardware_interface/PositionJointInterface</hardwareInterface>
-    </joint>
-  <actuator name="${name}_mirror2_roll_motor">
-      <hardwareInterface>hardware_interface/PositionJointInterface</hardwareInterface>
-      <mechanicalReduction>1</mechanicalReduction>
-    </actuator>
-  </transmission>
-  <transmission name="tran10">
-    <type>transmission_interface/SimpleTransmission</type>
-    <joint name="${name}_mirror1_prismatic_joint">
-      <hardwareInterface>hardware_interface/PositionJointInterface</hardwareInterface>
-    </joint>
-    <actuator name="${name}_mirror1_prismatic_motor">
-      <hardwareInterface>hardware_interface/PositionJointInterface</hardwareInterface>
-      <mechanicalReduction>1</mechanicalReduction>
-    </actuator>
-  </transmission>
-  <transmission name="tran11">
-    <type>transmission_interface/SimpleTransmission</type>
-    <joint name="${name}_mirror2_prismatic_joint">
-      <hardwareInterface>hardware_interface/PositionJointInterface</hardwareInterface>
-    </joint>
-    <actuator name="${name}_mirror2_prismatic_motor">
-      <hardwareInterface>hardware_interface/PositionJointInterface</hardwareInterface>
-      <mechanicalReduction>1</mechanicalReduction>
-    </actuator>
-  </transmission>
-  <transmission name="tran12">
-    <type>transmission_interface/SimpleTransmission</type>
-    <joint name="${name}_mirror1_prismatic2_joint">
-      <hardwareInterface>hardware_interface/PositionJointInterface</hardwareInterface>
-    </joint>
-    <actuator name="${name}_mirror1_prismatic2_motor">
-      <hardwareInterface>hardware_interface/PositionJointInterface</hardwareInterface>
-      <mechanicalReduction>1</mechanicalReduction>
-    </actuator>
-  </transmission>
-  <transmission name="tran13">
-    <type>transmission_interface/SimpleTransmission</type>
-    <joint name="${name}_mirror2_prismatic2_joint">
-      <hardwareInterface>hardware_interface/PositionJointInterface</hardwareInterface>
-    </joint>
-    <actuator name="${name}_mirror2_prismatic2_motor">
-      <hardwareInterface>hardware_interface/PositionJointInterface</hardwareInterface>
-      <mechanicalReduction>1</mechanicalReduction>
-    </actuator>
-  </transmission>
-  <transmission name="tran14">
-    <type>transmission_interface/SimpleTransmission</type>
-    <joint name="${name}_mirror1_pitch_joint">
-      <hardwareInterface>hardware_interface/PositionJointInterface</hardwareInterface>
-    </joint>
-  <actuator name="${name}_mirror1_pitch_motor">
-      <hardwareInterface>hardware_interface/PositionJointInterface</hardwareInterface>
-      <mechanicalReduction>1</mechanicalReduction>
-    </actuator>
-  </transmission>
-  <transmission name="tran15">
-    <type>transmission_interface/SimpleTransmission</type>
-    <joint name="${name}_mirror2_pitch_joint">
-      <hardwareInterface>hardware_interface/PositionJointInterface</hardwareInterface>
-    </joint>
-  <actuator name="${name}_mirror2_pitch_motor">
-      <hardwareInterface>hardware_interface/PositionJointInterface</hardwareInterface>
-      <mechanicalReduction>1</mechanicalReduction>
-    </actuator>
-  </transmission>
--->
-</xacro:macro>
+    <link name="${name}_right_prismatic2_link">
+      <inertial>
+        <origin xyz="0 0 0" />
+        <mass value="0.01" />
+        <inertia ixx="0.1" ixy="0.0" ixz="0.0" iyy="0.1" iyz="0.0" izz="0.1" />
+      </inertial>
+    </link>
+    <xacro:include filename="$(find icart_mini_description)/urdf/sensors/hokuyo.urdf.xacro"/>
+    <xacro:sensor_hokuyo name="${name}_right" parent="${name}_right_prismatic2_link">
+      <origin xyz="0 0 0" rpy="0 0 0"/>
+    </xacro:sensor_hokuyo>
+    <transmission name="${name}_left_roll_tran">
+      <type>transmission_interface/SimpleTransmission</type>
+      <joint name="${name}_left_roll_joint">
+        <hardwareInterface>hardware_interface/PositionJointInterface</hardwareInterface>
+      </joint>
+    <actuator name="${name}_left_roll_motor">
+        <hardwareInterface>hardware_interface/PositionJointInterface</hardwareInterface>
+        <mechanicalReduction>1</mechanicalReduction>
+      </actuator>
+    </transmission>
+    <transmission name="${name}_right_roll_tran">
+      <type>transmission_interface/SimpleTransmission</type>
+      <joint name="${name}_right_roll_joint">
+        <hardwareInterface>hardware_interface/PositionJointInterface</hardwareInterface>
+      </joint>
+    <actuator name="${name}_right_roll_motor">
+        <hardwareInterface>hardware_interface/PositionJointInterface</hardwareInterface>
+        <mechanicalReduction>1</mechanicalReduction>
+      </actuator>
+    </transmission>
+    <transmission name="${name}_left_prismatic_tran">
+      <type>transmission_interface/SimpleTransmission</type>
+      <joint name="${name}_left_prismatic_joint">
+        <hardwareInterface>hardware_interface/PositionJointInterface</hardwareInterface>
+      </joint>
+      <actuator name="${name}_left_prismatic_motor">
+        <hardwareInterface>hardware_interface/PositionJointInterface</hardwareInterface>
+        <mechanicalReduction>1</mechanicalReduction>
+      </actuator>
+    </transmission>
+    <transmission name="${name}_right_prismatic_tran">
+      <type>transmission_interface/SimpleTransmission</type>
+      <joint name="${name}_right_prismatic_joint">
+        <hardwareInterface>hardware_interface/PositionJointInterface</hardwareInterface>
+      </joint>
+      <actuator name="${name}_right_prismatic_motor">
+        <hardwareInterface>hardware_interface/PositionJointInterface</hardwareInterface>
+        <mechanicalReduction>1</mechanicalReduction>
+      </actuator>
+    </transmission>
+    <transmission name="{name}_left_prismatic2_tran">
+      <type>transmission_interface/SimpleTransmission</type>
+      <joint name="${name}_left_prismatic2_joint">
+        <hardwareInterface>hardware_interface/PositionJointInterface</hardwareInterface>
+      </joint>
+      <actuator name="${name}_left_prismatic2_motor">
+        <hardwareInterface>hardware_interface/PositionJointInterface</hardwareInterface>
+        <mechanicalReduction>1</mechanicalReduction>
+      </actuator>
+    </transmission>
+    <transmission name="${name}_right_prismatic2_tran">
+      <type>transmission_interface/SimpleTransmission</type>
+      <joint name="${name}_right_prismatic2_joint">
+        <hardwareInterface>hardware_interface/PositionJointInterface</hardwareInterface>
+      </joint>
+      <actuator name="${name}_right_prismatic2_motor">
+        <hardwareInterface>hardware_interface/PositionJointInterface</hardwareInterface>
+        <mechanicalReduction>1</mechanicalReduction>
+      </actuator>
+    </transmission>
+    <transmission name="${name}_left_pitch_tran">
+      <type>transmission_interface/SimpleTransmission</type>
+      <joint name="${name}_left_pitch_joint">
+        <hardwareInterface>hardware_interface/PositionJointInterface</hardwareInterface>
+      </joint>
+    <actuator name="${name}_left_pitch_motor">
+        <hardwareInterface>hardware_interface/PositionJointInterface</hardwareInterface>
+        <mechanicalReduction>1</mechanicalReduction>
+      </actuator>
+    </transmission>
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