Commit message: modify roll angle

File: lidar_with_mirror_description/urdf/sensor/lidar_with_mirror.urdf.xacro (robot description, xacro)
@@ -51,5 +51,5 @@
       <parent link="${name}_left_yaw_link"/>
       <child link="${name}_left_roll_link"/>
-      <origin xyz="0 0 0" rpy="${left_roll_rad} 0 0"/>
+      <origin xyz="0 0 0" rpy="${-left_roll_rad} 0 0"/>
       <axis xyz="1 0 0"/>
       <limit effort="100" velocity="100.0" lower="${-PI}" upper="${PI}" />
@@ -111,5 +111,5 @@
       <parent link="${name}_right_yaw_link"/>
       <child link="${name}_right_roll_link"/>
-      <origin xyz="0 0 0" rpy="-${right_roll_rad} 0 0"/>
+      <origin xyz="0 0 0" rpy="${right_roll_rad} 0 0"/>
       <axis xyz="-1 0 0"/>
       <limit effort="100" velocity="100.0" lower="${-PI}" upper="${PI}" />
